Commit message: add new robot model

File: legged_robot/tripod_3dof.urdf (robot description, URDF)
Before this commit: robot tripod, 7 links, 6 joints
Links:
- added link leg_0_3, mass 0.04; collision box size=0.025 0.025 0.14; collision sphere radius=0.025
- added link leg_2_3, mass 0.04; collision box size=0.025 0.025 0.14; collision sphere radius=0.025
- added link leg_4_3, mass 0.04; collision box size=0.025 0.025 0.14; collision sphere radius=0.025
Joints:
- added joint leg_0_2_3: type revolute, parent leg_0_2, child leg_0_3, origin xyz=0 0.085 0 rpy=-1.57079632679 0 0, axis -1 0 0, limit lower=-0.78539816339 upper=0.78539816339 effort=30.0 velocity=7.0
- added joint leg_2_2_3: type revolute, parent leg_2_2, child leg_2_3, origin xyz=0 0.085 0 rpy=-1.57079632679 0 0, axis -1 0 0, limit lower=-0.78539816339 upper=0.78539816339 effort=30.0 velocity=7.0
- added joint leg_4_2_3: type revolute, parent leg_4_2, child leg_4_3, origin xyz=0 -0.085 0 rpy=1.57079632679 0 0, axis 1 0 0, limit lower=-0.78539816339 upper=0.78539816339 effort=30.0 velocity=7.0

File: legged_robot/tripod_4dof.urdf (robot description, URDF)
Before this commit: robot tripod, 7 links, 6 joints
Links:
- added link leg_0_3, mass 0.184; collision box size=0.02 0.02 0.085; visual cylinder length=0.085 radius=0.02
- added link leg_0_4, mass 0.04; collision box size=0.025 0.025 0.14; collision sphere radius=0.025
- added link leg_2_3, mass 0.184; collision box size=0.02 0.02 0.085; visual cylinder length=0.085 radius=0.02
- added link leg_2_4, mass 0.04; collision box size=0.025 0.025 0.14; collision sphere radius=0.025
- added link leg_4_3, mass 0.184; collision box size=0.02 0.02 0.085; visual cylinder length=0.085 radius=0.02
- added link leg_4_4, mass 0.04; collision box size=0.025 0.025 0.14; collision sphere radius=0.025
Joints:
- added joint leg_0_2_3: type revolute, parent leg_0_2, child leg_0_3, origin xyz=0 0.085 0 rpy=0 0 0, axis 1 0 0, limit lower=-0.78539816339 upper=0.78539816339 effort=30.0 velocity=7.0
- added joint leg_0_3_4: type revolute, parent leg_0_3, child leg_0_4, origin xyz=0 0.085 0 rpy=-1.57079632679 0 0, axis -1 0 0, limit lower=-0.78539816339 upper=0.78539816339 effort=30.0 velocity=7.0
- added joint leg_2_2_3: type revolute, parent leg_2_2, child leg_2_3, origin xyz=0 0.085 0 rpy=0 0 0, axis 1 0 0, limit lower=-0.78539816339 upper=0.78539816339 effort=30.0 velocity=7.0
- added joint leg_2_3_4: type revolute, parent leg_2_3, child leg_2_4, origin xyz=0 0.085 0 rpy=-1.57079632679 0 0, axis -1 0 0, limit lower=-0.78539816339 upper=0.78539816339 effort=30.0 velocity=7.0
- added joint leg_4_2_3: type revolute, parent leg_4_2, child leg_4_3, origin xyz=0 -0.085 0 rpy=0 0 0, axis -1 0 0, limit lower=-0.78539816339 upper=0.78539816339 effort=30.0 velocity=7.0
- added joint leg_4_3_4: type revolute, parent leg_4_3, child leg_4_4, origin xyz=0 -0.085 0 rpy=1.57079632679 0 0, axis 1 0 0, limit lower=-0.78539816339 upper=0.78539816339 effort=30.0 velocity=7.0
